File: GR8RAM.kicad_pcb (KiCad board)
At the start: 4 copper layers, 99.9 x 59.8 mm, 69 parts, among them J1 AppleIIBus, J2 JTAG, J4 JTAG, J5 JTAG, SW1 FW, U1 EPM240T100C5N, U13 25M, U14 74LVC1G125GW, U16 74LVC1G125GW, U2 W9825, U3 W25Q128JVSIQ, U4 74AHC245PW, U5 74AHC245PW, U6 74AHC245PW, U8 XC6206P332MR, U9 74AHC245PW

Commit message: Add "ZK, GF" to board
Other:
- board text added: "ZK, GF"
Changed lines of the file:
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@@
   (general
     (thickness 1.6)
-    (drawings 57)
+    (drawings 58)
     (tracks 2386)
     (zones 0)
@@
     )
   )
+  (gr_text "ZK, GF" (at 132.461 129.921) (layer B.SilkS)
+    (effects (font (size 0.8128 0.8128) (thickness 0.2032)) (justify mirror))
+  )
   (gr_line (start 130.81 108.458) (end 129.032 108.458) (layer F.SilkS) (width 0.2032))
